File: 694200101R1/6942000101R1_sheet_2.sch (KiCad schematic (older format))
At the start: 89 parts

Commit message: Added B LED Driver and Initial plate deisgn
Added Second LED Array
Added DXF from ai03 and cusomized one for the volume/mute knob cut out
Parts:
- D? (x64): symbol 19-337C_RSBHGHC-A88_4T:19-337C_RSBHGHC-A88_4T -> 694200101-rescue:19-337C_RSBHGHC-A88_4T-19-337C_RSBHGHC-A88_4T

Commit message: Added 3D Models
Added 3D Models for all components
Added Keyboard DXF for reference
Parts:
- C10, C11, C12, C19, C20, C21, C22, C9: renamed from C?; footprint CAPC1608X90N -> capacitor-lib:CAPC1608X90N
- C13, C14, C15, C16, C17, C18: renamed from C?; footprint Samsung-CL10-09_2006-0-* -> capacitor-lib:Samsung-CL10-09_2006-0-IPC_C
- C23, C8: renamed from C?; footprint CAPPC3528X210N -> capacitor-lib:CAPPC3528X210N
- D104, D105, D106, D107, D108, D109, D110, D111, D112, D113, D114, D115, D116, D117, D118, D119, D120, D121, D122, D123, D124, D125, D126, D127, D128, D129, D130, D131, D132, D133, D134, D135, D136, D137, D138, D139, D140, D141, D142, D143, D144, D145, D146, D147, D148, D149, D150, D151, D152, D153, D154, D155, D156, D157, D158, D159, D160, D161, D162, D163, D164, D165, D166, D167: renamed from D?; footprint LED_19-337C/RSBHGHC-A88/4T -> RSBHGHC-A88:4T; symbol 694200101-rescue:19-337C_RSBHGHC-A88_4T-19-337C_RSBHGHC-A88_4T -> 19-337C_RSBHGHC-A88_4T:RGB_LED
- R10, R12, R13, R9: renamed from R?; footprint RESC1508X55N -> Resistor-Libs:RESC1508X55N
- R11, R14: renamed from R?; footprint RESC6332X70N -> Resistor-Libs:RESC6332X70N
- U3: renamed from U?; footprint STMicroelectronics-SO8N-SO-A-0-2-* -> STM:STMicroelectronics-SO8N-SO-A-0-2-IPC_C
- U4, U5: renamed from U?; footprint QFN-48_ISI -> Lumissil:IS31FL3733B-QFLS4-TR
