File: 694200101R1/694200101R1_sheet_3.sch (KiCad schematic (older format))
At the start: 48 parts

Commit message: top row buttons
Parts:
- renumbered D168 to D173, D169 to D174, D170 to D175, D171 to D176, D172 to D177, D173 to D178, D174 to D179, D175 to D180, D176 to D181, D177 to D182, D178 to D183, D179 to D184, D180 to D185, D181 to D186, D182 to D187, D183 to D188, D184 to D189, D185 to D190, D186 to D191, D187 to D192, D188 to D193, D189 to D194, D190 to D195, D191 to D196, D192 to D197, D193 to D198, D194 to D199, D195 to D200, D196 to D201, D197 to D202, D198 to D203, D199 to D204, D200 to D205, D201 to D206, D202 to D207, D203 to D208, D204 to D209, D205 to D210, D206 to D211, D207 to D212, D208 to D213, D209 to D214, D210 to D215, D211 to D216, D212 to D217, D213 to D218, D214 to D219, D215 to D220
