File: 694200101R1/694200101.sch (KiCad schematic (older format))
At the start: 255 parts, among them J1 USB4085-GF-A, J2 Conn_01x05_Male, J3 Conn_01x02_Male, SW1 MX_SW, SW10 MX_SW, SW100 MX_SW, SW101 MX_SW, SW102 MX_SW, SW103 MX_SW, SW104 MX_SW, SW105 MX_SW, SW106 MX_SW, SW107 MX_SW, SW11 MX_SW, SW12 MX_SW, SW13 MX_SW, SW14 MX_SW, SW15 MX_SW, SW16 MX_SW, SW17 MX_SW, SW18 MX_SW, SW19 MX_SW, SW2 MX_SW, SW20 MX_SW, SW21 MX_SW, SW22 MX_SW, SW23 MX_SW, SW24 MX_SW, SW25 MX_SW, SW26 MX_SW, SW27 MX_SW, SW28 MX_SW, SW29 MX_SW, SW3 MX_SW, SW30 MX_SW, SW31 MX_SW, SW32 MX_SW, SW33 MX_SW, SW34 MX_SW, SW35 MX_SW, SW36 MX_SW, SW37 MX_SW, SW38 MX_SW, SW39 MX_SW, SW4 MX_SW, SW40 MX_SW, SW41 MX_SW, SW42 MX_SW, SW43 MX_SW, SW44 MX_SW, SW45 MX_SW, SW46 MX_SW, SW47 MX_SW, SW48 MX_SW, SW49 MX_SW, SW5 MX_SW, SW50 MX_SW, SW51 MX_SW, SW52 MX_SW, SW53 MX_SW, SW54 MX_SW, SW55 MX_SW, SW56 MX_SW, SW57 MX_SW, SW58 MX_SW, SW59 MX_SW, SW6 MX_SW, SW60 MX_SW, SW61 MX_SW, SW62 MX_SW, SW63 MX_SW, SW64 MX_SW, SW65 MX_SW, SW66 MX_SW, SW67 MX_SW, SW68 MX_SW, SW69 MX_SW, SW7 MX_SW, SW70 MX_SW, SW71 MX_SW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

Commit message: usb traces
Parts:
- removed R?: RMCF0805FT510R, Resistor-Libs:RESC2012X65N, symbol Resistor-Lib:RMCF0805FT510R
- added R4: RMCF0805FT510R, Resistor-Libs:RESC2012X65N, symbol Resistor-Lib:RMCF0805FT510R
- gave numbers to parts that had none: 5
- renumbered C4 to C3, C3 to C4, R4 to R10, R5 to R11, R6 to R12, R7 to R13, R8 to R14, R3 to R9
Connections:
- net ROW_1: now also U3.56 (PB4)
- net ROW_2: now also R4.1; no longer U3.9 (PC1)
- new net: R4.2, U3.9 (PC1)
Changed lines of the file:
@@
 $EndComp
 $Comp
-L capacitor-lib:CL10B104KB8NNNL C3
+L capacitor-lib:CL10B104KB8NNNL C4
 U 1 1 5FFC635A
 P 5950 9700
-F 0 "C3" H 6078 9646 50  0000 L CNN
+F 0 "C4" H 6078 9646 50  0000 L CNN
 F 1 "CL10B104KB8NNNL" H 6078 9555 50  0001 L CNN
 F 2 "capacitor-lib:Samsung-CL10-09_2006-0-IPC_C" H 5950 10000 50  0001 L CNN
@@
 Connection ~ 5550 9600
 $Comp
-L power:+3V3 #PWR07
+L power:+3V3 #PWR08
 U 1 1 60025455
 P 6450 9600
-F 0 "#PWR07" H 6450 9450 50  0001 C CNN
+F 0 "#PWR08" H 6450 9450 50  0001 C CNN
 F 1 "+3V3" H 6465 9773 50  0000 C CNN
 F 2 "" H 6450 9600 50  0001 C CNN
@@
 Connection ~ 2950 9950
 $Comp
-L power:+3V3 #PWR012
+L power:+3V3 #PWR013
 U 1 1 6002F4CC
 P 8950 5950
-F 0 "#PWR012" H 8950 5800 50  0001 C CNN
+F 0 "#PWR013" H 8950 5800 50  0001 C CNN
 F 1 "+3V3" H 8965 6123 50  0000 C CNN
 F 2 "" H 8950 5950 50  0001 C CNN
@@
 Connection ~ 8950 10100
 $Comp
-L power:GND #PWR011
+L power:GND #PWR012
 U 1 1 5FFAF2AA
 P 8850 10200
-F 0 "#PWR011" H 8850 9950 50  0001 C CNN
+F 0 "#PWR012" H 8850 9950 50  0001 C CNN
 F 1 "GND" H 8772 10163 50  0000 R CNN
 F 2 "" H 8850 10200 50  0001 C CNN
@@
 $EndComp
 $Comp
-L power:+3V3 #PWR010
+L power:+3V3 #PWR09
 U 1 1 60076D41
 P 7750 7800
-F 0 "#PWR010" H 7750 7650 50  0001 C CNN
+F 0 "#PWR09" H 7750 7650 50  0001 C CNN
 F 1 "+3V3" H 7765 7973 50  0000 C CNN
 F 2 "" H 7750 7800 50  0001 C CNN
@@
 	8250 6600 7950 6600
 $Comp
-L power:GND #PWR09
+L power:GND #PWR010
 U 1 1 6007927B
 P 7950 6950
-F 0 "#PWR09" H 7950 6700 50  0001 C CNN
+F 0 "#PWR010" H 7950 6700 50  0001 C CNN
 F 1 "GND" H 7955 6777 50  0000 C CNN
 F 2 "" H 7950 6950 50  0001 C CNN
@@
 	15400 6500 15400 6350
 $Comp
-L Resistor-Lib:RNCP0603FTD10K0 R7
+L Resistor-Lib:RNCP0603FTD10K0 R13
 U 1 1 5FECBF04
 P 16050 6900
-F 0 "R7" V 16004 7005 50  0000 L CNN
+F 0 "R13" V 16004 7005 50  0000 L CNN
 F 1 "RNCP0603FTD10K0" H 15750 6700 50  0001 L BNN
 F 2 "Resistor-Libs:RESC1508X50N" H 16050 6900 50  0001 L BNN
@@
 $EndComp
 $Comp
-L Resistor-Lib:RNCP0603FTD10K0 R5
+L Resistor-Lib:RNCP0603FTD10K0 R11
 U 1 1 5FECA545
 P 15400 6900
-F 0 "R5" V 15354 7005 50  0000 L CNN
+F 0 "R11" V 15354 7005 50  0000 L CNN
 F 1 "RNCP0603FTD10K0" H 15100 6700 50  0001 L BNN
 F 2 "Resistor-Libs:RESC1508X50N" H 15400 6900 50  0001 L BNN
@@
 $EndComp
 $Comp
-L power:+3V3 #PWR015
+L power:+3V3 #PWR016
 U 1 1 5FEB4721
 P 15750 6350
-F 0 "#PWR015" H 15750 6200 50  0001 C CNN
+F 0 "#PWR016" H 15750 6200 50  0001 C CNN
 F 1 "+3V3" H 15765 6523 50  0000 C CNN
 F 2 "" H 15750 6350 50  0001 C CNN
@@
 Connection ~ 15400 7300
 $Comp
-L Resistor-Lib:RNCP0603FTD10K0 R6
+L Resistor-Lib:RNCP0603FTD10K0 R12
 U 1 1 5FF01719
 P 15400 7900
-F 0 "R6" V 15354 8005 50  0000 L CNN
+F 0 "R12" V 15354 8005 50  0000 L CNN
 F 1 "RNCP0603FTD10K0" H 15100 7700 50  0001 L BNN
 F 2 "Resistor-Libs:RESC1508X50N" H 15400 7900 50  0001 L BNN
@@
 $EndComp
 $Comp
-L Resistor-Lib:RNCP0603FTD10K0 R8
+L Resistor-Lib:RNCP0603FTD10K0 R14
 U 1 1 5FF03334
 P 16050 7900
-F 0 "R8" V 16004 8005 50  0000 L CNN
+F 0 "R14" V 16004 8005 50  0000 L CNN
 F 1 "RNCP0603FTD10K0" H 15750 7700 50  0001 L BNN
 F 2 "Resistor-Libs:RESC1508X50N" H 16050 7900 50  0001 L BNN
@@
 ENCODER_B
 $Comp
-L Resistor-Lib:RMCF0603FT1K00 R3
+L Resistor-Lib:RMCF0603FT1K00 R9
 U 1 1 6001106E
 P 11050 8450
-F 0 "R3" V 11004 8555 50  0000 L CNN
+F 0 "R9" V 11004 8555 50  0000 L CNN
 F 1 "RMCF0603FT1K00" V 11095 8555 50  0001 L CNN
 F 2 "Resistor-Libs:RESC1508X55N" H 11050 8450 50  0001 L BNN
@@
 $EndComp
 $Comp
-L Resistor-Lib:RMCF0603FT1K00 R4
+L Resistor-Lib:RMCF0603FT1K00 R10
 U 1 1 60013A68
 P 11300 8450
-F 0 "R4" V 11254 8555 50  0000 L CNN
+F 0 "R10" V 11254 8555 50  0000 L CNN
 F 1 "RMCF0603FT1K00" V 11345 8555 50  0001 L CNN
 F 2 "Resistor-Libs:RESC1508X55N" H 11300 8450 50  0001 L BNN
@@
 	11300 8000 11300 8050
 $Comp
-L power:+3V3 #PWR013
+L power:+3V3 #PWR014
 U 1 1 60025E0E
 P 11200 8000
-F 0 "#PWR013" H 11200 7850 50  0001 C CNN
+F 0 "#PWR014" H 11200 7850 50  0001 C CNN
 F 1 "+3V3" H 11215 8173 50  0000 C CNN
 F 2 "" H 11200 8000 50  0001 C CNN
@@
 Text GLabel 11400 7350 2    50   Input ~ 0
 ROW_0
-Text GLabel 11400 7100 2    50   Input ~ 0
+Text GLabel 9950 8700 2    50   Input ~ 0
 ROW_1
-Text GLabel 7900 8400 0    50   Input ~ 0
-ROW_2
 Wire Wire Line
 	8250 8100 7750 8100
@@
 COL_22
 $Comp
-L power:GND #PWR014
+L power:GND #PWR015
 U 1 1 5FEB2ECC
 P 14100 7900
-F 0 "#PWR014" H 14100 7650 50  0001 C CNN
+F 0 "#PWR015" H 14100 7650 50  0001 C CNN
 F 1 "GND" H 14105 7727 50  0000 C CNN
 F 2 "" H 14100 7900 50  0001 C CNN
@@
 $EndComp
 $Comp
-L capacitor-lib:06035A100JAT2A C4
+L capacitor-lib:06035A100JAT2A C3
 U 1 1 60087526
 P 5600 7500
-F 0 "C4" H 5727 7354 50  0000 L CNN
+F 0 "C3" H 5727 7354 50  0000 L CNN
 F 1 "06035A100JAT2A" H 5727 7445 50  0000 L CNN
 F 2 "capacitor-lib:AVX-GRM124-0-0-IPC_C" H 5600 7800 50  0001 L CNN
@@
 	7900 7700 8250 7700
 $Comp
-L power:GND #PWR08
+L power:GND #PWR07
 U 1 1 6065E993
 P 5600 7650
-F 0 "#PWR08" H 5600 7400 50  0001 C CNN
+F 0 "#PWR07" H 5600 7400 50  0001 C CNN
 F 1 "GND" H 5605 7477 50  0000 C CNN
 F 2 "" H 5600 7650 50  0001 C CNN
@@
 	1    0    0    -1
 $EndComp
-Wire Wire Line
-	8250 8400 7900 8400
 Text GLabel 10100 8600 2    50   Input ~ 0
 SWO
@@
 	8050 6050 8050 6100
 $Comp
-L power:GND #PWR0101
+L power:GND #PWR011
 U 1 1 602A2E5A
 P 8050 6100
-F 0 "#PWR0101" H 8050 5850 50  0001 C CNN
+F 0 "#PWR011" H 8050 5850 50  0001 C CNN
 F 1 "GND" H 8055 5927 50  0000 C CNN
 F 2 "" H 8050 6100 50  0001 C CNN
@@
 	9550 7200 9900 7200
 Wire Wire Line
-	10450 8700 10450 7100
-Wire Wire Line
-	9550 8700 10450 8700
-Wire Wire Line
 	10500 8800 10500 7350
 Wire Wire Line
@@
 	9550 8800 10500 8800
 Wire Wire Line
-	10450 7100 10550 7100
-$Comp
-L Resistor-Lib:RMCF0805FT510R R?
-U 1 1 61756588
-P 10950 7100
-F 0 "R?" H 10650 7150 50  0000 C CNN
-F 1 "RMCF0805FT510R" H 10650 6850 50  0001 L BNN
-F 2 "Resistor-Libs:RESC2012X65N" H 10650 6950 50  0001 L BNN
-F 3 "" H 10950 7100 50  0001 L BNN
-F 4 "510" H 11250 7150 50  0000 C CNN "reistance"
-	1    10950 7100
-	1    0    0    -1
-$EndComp
-Wire Wire Line
-	11350 7100 11400 7100
-Wire Wire Line
 	11400 7350 11350 7350
 $Comp
-L Resistor-Lib:RMCF0805FT510R R?
+L Resistor-Lib:RMCF0805FT510R R8
 U 1 1 6183038F
 P 10950 7350
-F 0 "R?" H 10650 7400 50  0000 C CNN
+F 0 "R8" H 10650 7400 50  0000 C CNN
 F 1 "RMCF0805FT510R" H 10650 7100 50  0001 L BNN
 F 2 "Resistor-Libs:RESC2012X65N" H 10650 7200 50  0001 L BNN
@@
 $EndComp
 $Comp
-L Resistor-Lib:RMCF0805FT510R R?
+L Resistor-Lib:RMCF0805FT510R R3
 U 1 1 61907867
 P 7350 8100
-F 0 "R?" H 7350 8342 50  0000 C CNN
+F 0 "R3" H 7350 8342 50  0000 C CNN
 F 1 "RMCF0805FT510R" H 7050 7850 50  0001 L BNN
 F 2 "Resistor-Libs:RESC2012X65N" H 7050 7950 50  0001 L BNN
@@
 	8150 10300 8000 10300
 $Comp
-L Resistor-Lib:RMCF0805FT510R R?
+L Resistor-Lib:RMCF0805FT510R R7
 U 1 1 61BF657B
 P 7600 10300
-F 0 "R?" H 7300 10350 50  0000 C CNN
+F 0 "R7" H 7300 10350 50  0000 C CNN
 F 1 "RMCF0805FT510R" H 7300 10050 50  0001 L BNN
 F 2 "Resistor-Libs:RESC2012X65N" H 7300 10150 50  0001 L BNN
@@
 	7150 10300 7200 10300
 $Comp
-L Resistor-Lib:RMCF0805FT510R R?
+L Resistor-Lib:RMCF0805FT510R R6
 U 1 1 61C65077
 P 7600 10100
-F 0 "R?" H 7300 10150 50  0000 C CNN
+F 0 "R6" H 7300 10150 50  0000 C CNN
 F 1 "RMCF0805FT510R" H 7300 9850 50  0001 L BNN
 F 2 "Resistor-Libs:RESC2012X65N" H 7300 9950 50  0001 L BNN
@@
 	8000 9300 8000 9900
 $Comp
-L Resistor-Lib:RMCF0805FT510R R?
+L Resistor-Lib:RMCF0805FT510R R5
 U 1 1 61E7DED3
 P 7600 9900
-F 0 "R?" H 7300 9950 50  0000 C CNN
+F 0 "R5" H 7300 9950 50  0000 C CNN
 F 1 "RMCF0805FT510R" H 7300 9650 50  0001 L BNN
 F 2 "Resistor-Libs:RESC2012X65N" H 7300 9750 50  0001 L BNN
@@
 	1    0    0    -1
 $EndComp
+Wire Wire Line
+	9550 8700 9950 8700
+$Comp
+L Resistor-Lib:RMCF0805FT510R R4
+U 1 1 602BDFC6
+P 7350 8400
+F 0 "R4" H 7050 8450 50  0000 C CNN
+F 1 "RMCF0805FT510R" H 7050 8150 50  0001 L BNN
+F 2 "Resistor-Libs:RESC2012X65N" H 7050 8250 50  0001 L BNN
+F 3 "" H 7350 8400 50  0001 L BNN
+F 4 "510" H 7650 8450 50  0000 C CNN "reistance"
+	1    7350 8400
+	1    0    0    -1
+$EndComp
+Text GLabel 6900 8400 0    50   Input ~ 0
+ROW_2
+Wire Wire Line
+	7750 8400 8250 8400
+Wire Wire Line
+	6950 8400 6900 8400
 $EndSCHEMATC
