File: 694200101R1/694200101R1_sheet_2.sch (KiCad schematic (older format))
At the start: 89 parts, among them U4 M24M02-DRMN6TP, U5 IS31FL3733B-QFLS4-TR, U6 IS31FL3733B-QFLS4-TR

Commit message: usb traces
Parts:
- renumbered R9 to R15, R10 to R16, R11 to R17, R12 to R18, R13 to R19, R14 to R20
Changed lines of the file:
@@
 $EndComp
 $Comp
-L power:+3V3 #PWR016
+L power:+3V3 #PWR017
 U 1 1 63D43A95
 P 1500 7600
-F 0 "#PWR016" H 1500 7450 50  0001 C CNN
+F 0 "#PWR017" H 1500 7450 50  0001 C CNN
 F 1 "+3V3" H 1515 7773 50  0000 C CNN
 F 2 "" H 1500 7600 50  0001 C CNN
@@
 $EndComp
 $Comp
-L power:GND #PWR017
+L power:GND #PWR018
 U 1 1 63D489E9
 P 2550 8500
-F 0 "#PWR017" H 2550 8250 50  0001 C CNN
+F 0 "#PWR018" H 2550 8250 50  0001 C CNN
 F 1 "GND" H 2555 8327 50  0000 C CNN
 F 2 "" H 2550 8500 50  0001 C CNN
@@
 $EndComp
 $Comp
-L power:+3V3 #PWR028
+L power:+3V3 #PWR029
 U 1 1 63D70980
 P 13100 6800
-F 0 "#PWR028" H 13100 6650 50  0001 C CNN
+F 0 "#PWR029" H 13100 6650 50  0001 C CNN
 F 1 "+3V3" H 13115 6973 50  0000 C CNN
 F 2 "" H 13100 6800 50  0001 C CNN
@@
 $EndComp
 $Comp
-L power:GND #PWR029
+L power:GND #PWR030
 U 1 1 63D793EB
 P 13100 7250
-F 0 "#PWR029" H 13100 7000 50  0001 C CNN
+F 0 "#PWR030" H 13100 7000 50  0001 C CNN
 F 1 "GND" H 13105 7077 50  0000 C CNN
 F 2 "" H 13100 7250 50  0001 C CNN
@@
 $EndComp
 $Comp
-L power:+3V3 #PWR019
+L power:+3V3 #PWR020
 U 1 1 63D94BE2
 P 3600 8900
-F 0 "#PWR019" H 3600 8750 50  0001 C CNN
+F 0 "#PWR020" H 3600 8750 50  0001 C CNN
 F 1 "+3V3" H 3615 9073 50  0000 C CNN
 F 2 "" H 3600 8900 50  0001 C CNN
@@
 $EndComp
 $Comp
-L Resistor-Lib:RMCF0603FT100K R10
+L Resistor-Lib:RMCF0603FT100K R16
 U 1 1 63EAB8BE
 P 2800 9650
-F 0 "R10" V 2754 9755 50  0000 L CNN
+F 0 "R16" V 2754 9755 50  0000 L CNN
 F 1 "RMCF0603FT100K" H 2500 9450 50  0001 L BNN
 F 2 "Resistor-Libs:RESC1508X55N" H 2800 9650 50  0001 L BNN
@@
 $EndComp
 $Comp
-L Resistor-Lib:RMCF0603FT100K R9
+L Resistor-Lib:RMCF0603FT100K R15
 U 1 1 63EB01BF
 P 2600 9650
-F 0 "R9" V 2554 9546 50  0000 R CNN
+F 0 "R15" V 2554 9546 50  0000 R CNN
 F 1 "RMCF0603FT100K" H 2300 9450 50  0001 L BNN
 F 2 "Resistor-Libs:RESC1508X55N" H 2600 9650 50  0001 L BNN
@@
 $EndComp
 $Comp
-L power:GND #PWR018
+L power:GND #PWR019
 U 1 1 63EC1EB0
 P 3000 10150
-F 0 "#PWR018" H 3000 9900 50  0001 C CNN
+F 0 "#PWR019" H 3000 9900 50  0001 C CNN
 F 1 "GND" H 3005 9977 50  0000 C CNN
 F 2 "" H 3000 10150 50  0001 C CNN
@@
 $EndComp
 $Comp
-L Resistor-Lib:RMCF2512FT20K0 R11
+L Resistor-Lib:RMCF2512FT20K0 R17
 U 1 1 63ED9B4F
 P 3200 9650
-F 0 "R11" V 3154 9755 50  0000 L CNN
+F 0 "R17" V 3154 9755 50  0000 L CNN
 F 1 "RMCF2512FT20K0" H 2900 9450 50  0001 L BNN
 F 2 "Resistor-Libs:RESC6332X70N" H 3200 9650 50  0001 L BNN
@@
 $EndComp
 $Comp
-L power:GND #PWR020
+L power:GND #PWR021
 U 1 1 63EFD874
 P 3750 8250
-F 0 "#PWR020" H 3750 8000 50  0001 C CNN
+F 0 "#PWR021" H 3750 8000 50  0001 C CNN
 F 1 "GND" H 3755 8077 50  0000 C CNN
 F 2 "" H 3750 8250 50  0001 C CNN
@@
 $EndComp
 $Comp
-L power:+3V3 #PWR024
+L power:+3V3 #PWR025
 U 1 1 6409AB1B
 P 7700 8900
-F 0 "#PWR024" H 7700 8750 50  0001 C CNN
+F 0 "#PWR025" H 7700 8750 50  0001 C CNN
 F 1 "+3V3" H 7715 9073 50  0000 C CNN
 F 2 "" H 7700 8900 50  0001 C CNN
@@
 $EndComp
 $Comp
-L Resistor-Lib:RMCF0603FT100K R13
+L Resistor-Lib:RMCF0603FT100K R19
 U 1 1 6409AB23
 P 6900 9650
-F 0 "R13" V 6854 9755 50  0000 L CNN
+F 0 "R19" V 6854 9755 50  0000 L CNN
 F 1 "RMCF0603FT100K" H 6600 9450 50  0001 L BNN
 F 2 "Resistor-Libs:RESC1508X55N" H 6900 9650 50  0001 L BNN
@@
 $EndComp
 $Comp
-L Resistor-Lib:RMCF0603FT100K R12
+L Resistor-Lib:RMCF0603FT100K R18
 U 1 1 6409AB2A
 P 6700 9650
-F 0 "R12" V 6654 9546 50  0000 R CNN
+F 0 "R18" V 6654 9546 50  0000 R CNN
 F 1 "RMCF0603FT100K" H 6400 9450 50  0001 L BNN
 F 2 "Resistor-Libs:RESC1508X55N" H 6700 9650 50  0001 L BNN
@@
 $EndComp
 $Comp
-L power:GND #PWR023
+L power:GND #PWR024
 U 1 1 6409AB40
 P 7100 10150
-F 0 "#PWR023" H 7100 9900 50  0001 C CNN
+F 0 "#PWR024" H 7100 9900 50  0001 C CNN
 F 1 "GND" H 7105 9977 50  0000 C CNN
 F 2 "" H 7100 10150 50  0001 C CNN
@@
 $EndComp
 $Comp
-L Resistor-Lib:RMCF2512FT20K0 R14
+L Resistor-Lib:RMCF2512FT20K0 R20
 U 1 1 6409AB49
 P 7300 9650
-F 0 "R14" V 7254 9755 50  0000 L CNN
+F 0 "R20" V 7254 9755 50  0000 L CNN
 F 1 "RMCF2512FT20K0" H 7000 9450 50  0001 L BNN
 F 2 "Resistor-Libs:RESC6332X70N" H 7300 9650 50  0001 L BNN
@@
 $EndComp
 $Comp
-L power:GND #PWR025
+L power:GND #PWR026
 U 1 1 6409AB59
 P 7850 8250
-F 0 "#PWR025" H 7850 8000 50  0001 C CNN
+F 0 "#PWR026" H 7850 8000 50  0001 C CNN
 F 1 "GND" H 7855 8077 50  0000 C CNN
 F 2 "" H 7850 8250 50  0001 C CNN
@@
 $EndComp
 $Comp
-L power:+3V3 #PWR026
+L power:+3V3 #PWR027
 U 1 1 6409AB74
 P 10350 9600
-F 0 "#PWR026" H 10350 9450 50  0001 C CNN
+F 0 "#PWR027" H 10350 9450 50  0001 C CNN
 F 1 "+3V3" H 10365 9773 50  0000 C CNN
 F 2 "" H 10350 9600 50  0001 C CNN
@@
 $EndComp
 $Comp
-L power:GND #PWR027
+L power:GND #PWR028
 U 1 1 6409AB6A
 P 10400 8900
-F 0 "#PWR027" H 10400 8650 50  0001 C CNN
+F 0 "#PWR028" H 10400 8650 50  0001 C CNN
 F 1 "GND" H 10405 8727 50  0000 C CNN
 F 2 "" H 10400 8900 50  0001 C CNN
@@
 $EndComp
 $Comp
-L power:+3V3 #PWR021
+L power:+3V3 #PWR022
 U 1 1 63F20B48
 P 6250 9600
-F 0 "#PWR021" H 6250 9450 50  0001 C CNN
+F 0 "#PWR022" H 6250 9450 50  0001 C CNN
 F 1 "+3V3" H 6265 9773 50  0000 C CNN
 F 2 "" H 6250 9600 50  0001 C CNN
@@
 $EndComp
 $Comp
-L power:GND #PWR022
+L power:GND #PWR023
 U 1 1 63F0DD67
 P 6300 8900
-F 0 "#PWR022" H 6300 8650 50  0001 C CNN
+F 0 "#PWR023" H 6300 8650 50  0001 C CNN
 F 1 "GND" H 6305 8727 50  0000 C CNN
 F 2 "" H 6300 8900 50  0001 C CNN

Commit message: layout  led driver 1
Parts:
- removed C13, C24: CL10B474KA8NFNC, capacitor-lib:CAPC1608X90N, symbol capacitor-lib:CL10B474KA8NFNC
- renumbered C14 to C13, C15 to C14, C16 to C15, C17 to C16, C18 to C17, C19 to C18, C20 to C19, C21 to C20, C22 to C21, C23 to C22, C25 to C23, C26 to C24
Connections:
- net +3V3: no longer R16.1, R19.1, U5.46 (SDB), U6.46 (SDB)
- new net: R16.1, U5.46 (SDB)
- new net: R19.1, U6.46 (SDB)
Other:
- note removed: "LED_DRIVER_A\nP39"
- note removed: "LED_DRIVER_B\nP39"
Changed lines of the file:
@@
 Text Notes 10350 6850 1    50   ~ 0
 LED_DRIVER_A\nP37/38
-Wire Wire Line
-	10300 6900 10900 6900
 Connection ~ 10300 6900
-Wire Wire Line
-	10300 7250 10900 7250
-Wire Wire Line
-	10900 7250 10900 7200
-Wire Wire Line
-	10900 6900 11350 6900
-Connection ~ 10900 6900
 Connection ~ 11350 6900
 Wire Wire Line
@@
 Wire Wire Line
 	11550 7250 11350 7250
-Connection ~ 10900 7250
 Wire Wire Line
 	11350 7200 11350 7250
 Connection ~ 11350 7250
 Wire Wire Line
-	11350 7250 10900 7250
-Wire Wire Line
 	13100 6900 13100 6800
 Wire Wire Line
@@
 	12350 7250 12350 7150
 Connection ~ 12150 7250
-Text Notes 10950 6850 1    50   ~ 0
-LED_DRIVER_A\nP39
 Text Notes 11500 6850 1    50   ~ 0
 LED_DRIVER_A\nP20
@@
 Wire Wire Line
 	2800 8950 2800 9250
-Wire Wire Line
-	3400 8950 3600 8950
-Connection ~ 3400 8950
 Connection ~ 3600 8950
 Wire Wire Line
@@
 Wire Wire Line
 	6900 8950 6900 9250
-Wire Wire Line
-	7500 8950 7700 8950
-Connection ~ 7500 8950
 Connection ~ 7700 8950
 Wire Wire Line
@@
 $EndComp
 $Comp
-L capacitor-lib:CL10B474KA8NFNC C13
-U 1 1 63D81B26
-P 10900 7000
-F 0 "C13" V 11000 6850 50  0000 C CNN
-F 1 "CL10B474KA8NFNC" V 10995 7103 50  0001 L BNN
-F 2 "capacitor-lib:CAPC1608X90N" H 10900 7000 50  0001 L BNN
-F 3 "" H 10900 7000 50  0001 L BNN
-F 4 "https://pricing.snapeda.com/search/part/CL10B474KA8NFNC/?ref=eda" H 10900 7000 50  0001 L BNN "Purchase-URL"
-F 5 "0603 Samsung" H 10900 7000 50  0001 L BNN "Package"
-F 6 "CL10B474KA8NFNC" H 10900 7000 50  0001 L BNN "MP"
-F 7 "1276-2082-1-ND" H 10900 7000 50  0001 L BNN "Digi-Key_Part_Number"
-F 8 "Samsung Electro-Mechanics" H 10900 7000 50  0001 L BNN "MF"
-F 9 "0.47µF ±10% 25V Ceramic Capacitor X7R 0603 (1608 Metric)" H 10900 7000 50  0001 L BNN "Description"
-F 10 "0.47µF" V 11100 6850 50  0000 C CNN "capacitance"
-	1    10900 7000
-	0    1    1    0
-$EndComp
-$Comp
 L power:+3V3 #PWR020
 U 1 1 63D94BE2
@@
 $EndComp
 $Comp
-L capacitor-lib:CL10B474KA8NFNC C14
+L capacitor-lib:CL10B474KA8NFNC C13
 U 1 1 63D9DE47
 P 11350 7000
-F 0 "C14" V 11450 6850 50  0000 C CNN
+F 0 "C13" V 11450 6850 50  0000 C CNN
 F 1 "CL10B474KA8NFNC" H 11350 6800 50  0001 L BNN
 F 2 "capacitor-lib:CAPC1608X90N" H 11350 7000 50  0001 L BNN
@@
 $EndComp
 $Comp
-L capacitor-lib:CL10B104KB8NNNL C15
+L capacitor-lib:CL10B104KB8NNNL C14
 U 1 1 63D9F36F
 P 11550 6950
-F 0 "C15" H 11723 6850 50  0000 C CNN
+F 0 "C14" H 11723 6850 50  0000 C CNN
 F 1 "CL10B104KB8NNNL" H 11550 7150 50  0001 L CNN
 F 2 "capacitor-lib:Samsung-CL10-09_2006-0-IPC_C" H 11550 7250 50  0001 L CNN
@@
 $EndComp
 $Comp
-L capacitor-lib:CL10B474KA8NFNC C16
+L capacitor-lib:CL10B474KA8NFNC C15
 U 1 1 63DE9808
 P 12150 7000
-F 0 "C16" V 12250 7150 50  0000 C CNN
+F 0 "C15" V 12250 7150 50  0000 C CNN
 F 1 "CL10B474KA8NFNC" H 12150 6800 50  0001 L BNN
 F 2 "capacitor-lib:CAPC1608X90N" H 12150 7000 50  0001 L BNN
@@
 	10100 6900 10300 6900
 $Comp
-L capacitor-lib:TAJB226K016RNJ C18
+L capacitor-lib:TAJB226K016RNJ C17
 U 1 1 63E8E5AC
 P 12800 7100
-F 0 "C18" V 12850 6950 50  0000 C TNN
+F 0 "C17" V 12850 6950 50  0000 C TNN
 F 1 "TAJB226K016RNJ" H 12800 6900 50  0001 L BNN
 F 2 "capacitor-lib:CAPPC3528X210N" H 12800 7100 50  0001 L BNN
@@
 $EndComp
 $Comp
-L capacitor-lib:CL10B104KB8NNNL C17
+L capacitor-lib:CL10B104KB8NNNL C16
 U 1 1 63DECC4B
 P 12350 6950
-F 0 "C17" H 12523 6850 50  0000 C CNN
+F 0 "C16" H 12523 6850 50  0000 C CNN
 F 1 "CL10B104KB8NNNL" H 12350 7150 50  0001 L CNN
 F 2 "capacitor-lib:Samsung-CL10-09_2006-0-IPC_C" H 12350 7250 50  0001 L CNN
@@
 	16100 6900 15900 6900
 $Comp
-L capacitor-lib:CL10B474KA8NFNC C21
+L capacitor-lib:CL10B474KA8NFNC C20
 U 1 1 63E29468
 P 14050 7050
-F 0 "C21" V 14100 7200 50  0000 C CNN
+F 0 "C20" V 14100 7200 50  0000 C CNN
 F 1 "CL10B474KA8NFNC" H 14050 6850 50  0001 L BNN
 F 2 "capacitor-lib:CAPC1608X90N" H 14050 7050 50  0001 L BNN
@@
 $EndComp
 $Comp
-L capacitor-lib:CL10B104KB8NNNL C20
+L capacitor-lib:CL10B104KB8NNNL C19
 U 1 1 63E29486
 P 13850 7000
-F 0 "C20" H 14023 6900 50  0000 C CNN
+F 0 "C19" H 14023 6900 50  0000 C CNN
 F 1 "CL10B104KB8NNNL" H 13850 7200 50  0001 L CNN
 F 2 "capacitor-lib:Samsung-CL10-09_2006-0-IPC_C" H 13850 7300 50  0001 L CNN
@@
 $EndComp
 $Comp
-L capacitor-lib:CL10B104KB8NNNL C22
+L capacitor-lib:CL10B104KB8NNNL C21
 U 1 1 63E29448
 P 14650 7000
-F 0 "C22" H 14823 6900 50  0000 C CNN
+F 0 "C21" H 14823 6900 50  0000 C CNN
 F 1 "CL10B104KB8NNNL" H 14650 7200 50  0001 L CNN
 F 2 "capacitor-lib:Samsung-CL10-09_2006-0-IPC_C" H 14650 7300 50  0001 L CNN
@@
 $EndComp
 $Comp
-L capacitor-lib:CL10B474KA8NFNC C23
+L capacitor-lib:CL10B474KA8NFNC C22
 U 1 1 63E2942E
 P 14850 7050
-F 0 "C23" V 14900 6900 50  0000 C CNN
+F 0 "C22" V 14900 6900 50  0000 C CNN
 F 1 "CL10B474KA8NFNC" H 14850 6850 50  0001 L BNN
 F 2 "capacitor-lib:CAPC1608X90N" H 14850 7050 50  0001 L BNN
@@
 $EndComp
 $Comp
-L capacitor-lib:CL10B474KA8NFNC C24
-U 1 1 63E2941C
-P 15300 7050
-F 0 "C24" V 15350 6900 50  0000 C CNN
-F 1 "CL10B474KA8NFNC" V 15395 7153 50  0001 L BNN
-F 2 "capacitor-lib:CAPC1608X90N" H 15300 7050 50  0001 L BNN
-F 3 "" H 15300 7050 50  0001 L BNN
-F 4 "https://pricing.snapeda.com/search/part/CL10B474KA8NFNC/?ref=eda" H 15300 7050 50  0001 L BNN "Purchase-URL"
-F 5 "0603 Samsung" H 15300 7050 50  0001 L BNN "Package"
-F 6 "CL10B474KA8NFNC" H 15300 7050 50  0001 L BNN "MP"
-F 7 "1276-2082-1-ND" H 15300 7050 50  0001 L BNN "Digi-Key_Part_Number"
-F 8 "Samsung Electro-Mechanics" H 15300 7050 50  0001 L BNN "MF"
-F 9 "0.47µF ±10% 25V Ceramic Capacitor X7R 0603 (1608 Metric)" H 15300 7050 50  0001 L BNN "Description"
-F 10 "0.47µF" V 15450 6900 50  0000 C CNN "capacitance"
-	1    15300 7050
-	0    -1   1    0
-$EndComp
-$Comp
-L capacitor-lib:CL10B104KB8NNNL C25
+L capacitor-lib:CL10B104KB8NNNL C23
 U 1 1 63E2940D
 P 15900 7000
-F 0 "C25" H 16100 6900 50  0000 C CNN
+F 0 "C23" H 16100 6900 50  0000 C CNN
 F 1 "CL10B104KB8NNNL" H 16028 6900 50  0001 L CNN
 F 2 "capacitor-lib:Samsung-CL10-09_2006-0-IPC_C" H 15900 7300 50  0001 L CNN
@@
 Connection ~ 14850 7250
 Wire Wire Line
-	15300 7250 14850 7250
-Connection ~ 15300 7250
-Wire Wire Line
-	15900 7250 15300 7250
-Wire Wire Line
 	16100 7250 15900 7250
 Text Notes 14850 6850 1    50   ~ 0
 LED_DRIVER_B\nP29
-Text Notes 15350 6850 1    50   ~ 0
-LED_DRIVER_B\nP39
 Connection ~ 14050 6900
 Wire Wire Line
@@
 Wire Wire Line
 	14650 6900 14650 7000
-Wire Wire Line
-	14850 6900 15300 6900
 Connection ~ 14850 6900
 Wire Wire Line
 	14850 6950 14850 6900
-Connection ~ 15300 6900
 Wire Wire Line
 	14650 6900 14850 6900
-Wire Wire Line
-	15300 6900 15300 6950
-Wire Wire Line
-	15900 6900 15300 6900
 Connection ~ 15900 7250
 Text Notes 16000 6850 1    50   ~ 0
@@
 	15900 7250 15900 7200
 $Comp
-L capacitor-lib:CL10B474KA8NFNC C26
+L capacitor-lib:CL10B474KA8NFNC C24
 U 1 1 63E293F3
 P 16100 7050
-F 0 "C26" V 16150 6900 50  0000 C CNN
+F 0 "C24" V 16150 6900 50  0000 C CNN
 F 1 "CL10B474KA8NFNC" V 16195 7153 50  0001 L BNN
 F 2 "capacitor-lib:CAPC1608X90N" H 16100 7050 50  0001 L BNN
@@
 $EndComp
 $Comp
-L capacitor-lib:TAJB226K016RNJ C19
+L capacitor-lib:TAJB226K016RNJ C18
 U 1 1 63E9B64D
 P 13400 7100
-F 0 "C19" V 13450 6952 50  0000 C CNN
+F 0 "C18" V 13450 6952 50  0000 C CNN
 F 1 "TAJB226K016RNJ" H 13400 6900 50  0001 L BNN
 F 2 "capacitor-lib:CAPPC3528X210N" H 13400 7100 50  0001 L BNN
@@
 Wire Wire Line
 	3150 7000 7250 7000
+Wire Wire Line
+	10300 7250 11350 7250
+Wire Wire Line
+	10300 6900 11350 6900
+Wire Wire Line
+	14850 7250 15900 7250
+Wire Wire Line
+	14850 6900 15900 6900
 $EndSCHEMATC
