File: 694200101R1/694200101.kicad_pcb (KiCad board)
At the start: 2 copper layers, 438.6 x 125.8 mm, 395 parts, among them J1 USB4085-GF-A, J2 Conn_01x05_Male, J3 Conn_01x02_Male, SW1 MX_SW, SW10 MX_SW, SW100 MX_SW, SW101 MX_SW, SW102 MX_SW, SW103 MX_SW, SW104 MX_SW, SW105 MX_SW, SW106 MX_SW, SW107 MX_SW, SW11 MX_SW, SW12 MX_SW, SW13 MX_SW, SW14 MX_SW, SW15 MX_SW, SW16 MX_SW, SW17 MX_SW, SW18 MX_SW, SW19 MX_SW, SW2 MX_SW, SW20 MX_SW, SW21 MX_SW, SW22 MX_SW, SW23 MX_SW, SW24 MX_SW, SW25 MX_SW, SW26 MX_SW, SW27 MX_SW, SW28 MX_SW, SW29 MX_SW, SW3 MX_SW, SW30 MX_SW, SW31 MX_SW, SW32 MX_SW, SW33 MX_SW, SW34 MX_SW, SW35 MX_SW, SW36 MX_SW, SW37 MX_SW, SW38 MX_SW, SW39 MX_SW, SW4 MX_SW, SW40 MX_SW, SW41 MX_SW, SW42 MX_SW, SW43 MX_SW, SW44 MX_SW, SW45 MX_SW, SW46 MX_SW, SW47 MX_SW, SW48 MX_SW, SW49 MX_SW, SW5 MX_SW, SW50 MX_SW, SW51 MX_SW, SW52 MX_SW, SW53 MX_SW, SW54 MX_SW, SW55 MX_SW, SW56 MX_SW, SW57 MX_SW, SW58 MX_SW, SW59 MX_SW, SW6 MX_SW, SW60 MX_SW, SW61 MX_SW, SW62 MX_SW, SW63 MX_SW, SW64 MX_SW, SW65 MX_SW, SW66 MX_SW, SW67 MX_SW, SW68 MX_SW, SW69 MX_SW, SW7 MX_SW, SW70 MX_SW, SW71 MX_SW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

Commit message: cpoied second led driver
Parts:
- moved C24 21.7 mm to (386.0, -36.4), turned to 90 degrees
- moved C22 18.8 mm to (388.9, -29.0), turned to 270 degrees
- moved C19 15.7 mm to (384.6, -24.8), turned to 270 degrees
- moved C20 13.3 mm to (383.0, -24.6), turned to 270 degrees
- moved C6 11.8 mm to (356.5, 13.3), turned to 0 degrees
- moved C3 11.5 mm to (360.0, 16.1), turned to 90 degrees
- moved Y1 11.3 mm to (357.0, 16.0), turned to 180 degrees
- moved R19 9.47 mm to (378.3, -33.1), turned to 270 degrees
- moved C21 9.15 mm to (390.5, -29.0), turned to 270 degrees
- moved R18 9.10 mm to (376.8, -33.5), turned to 270 degrees
- moved C18 6.20 mm to (393.7, -28.6), turned to 270 degrees
- moved R10 2.84 mm to (349.2, 22.7)
- moved R4 2.84 mm to (360.7, 19.3)
- moved R9 2.84 mm to (347.7, 23.5)
- moved R3 2.84 mm to (355.0, 26.3)
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Routing:
- net ROW_0: track 301.6 -> 262.9 mm
- net Net-(C6-Pad1): track 0.00 -> 7.18 mm
- net Net-(C3-Pad1): track 0.00 -> 5.42 mm
- net GND: track 0.00 -> 3.09 mm

Commit message: led driver a layout pt1
Parts:
- C11, C12, C13, C14, C15, C16, C17, C18, C19, C20, C21, C22, C23, C24, R15, R16, R17, R18, R19, R20, U5, U6: moved to B.Cu
- moved C12 305.4 mm to (32.3, 24.5), turned to 270 degrees
- moved C11 305.4 mm to (33.9, 24.5), turned to 270 degrees
- moved R17 305.0 mm to (36.8, 24.5), turned to 270 degrees
- moved U5 303.5 mm to (30.7, 18.9)
- moved R15 302.8 mm to (27.9, 23.6), turned to 180 degrees
- moved C15 302.3 mm to (36.8, 17.5), turned to 90 degrees
- moved C16 302.3 mm to (38.5, 17.4), turned to 90 degrees
- moved C17 302.1 mm to (41.8, 16.8), turned to 90 degrees
- moved C13 301.7 mm to (31.2, 12.6), turned to 90 degrees
- moved C14 301.7 mm to (32.8, 12.6), turned to 90 degrees
- moved R16 299.0 mm to (30.6, 24.4), turned to 90 degrees
- moved R18 136.0 mm to (347.0, 99.2), turned to 180 degrees
- moved R19 134.6 mm to (346.6, 97.7), turned to 180 degrees
- moved C23 132.7 mm to (349.9, 91.7), turned to 0 degrees
- moved C24 131.5 mm to (349.9, 90.0), turned to 0 degrees
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Routing:
- net Net-(R16-Pad1): track 0.00 -> 4.25 mm
- net CS12_A: track 0.00 -> 2.01 mm
- net CS10_A: track 0.00 -> 1.98 mm
- net Net-(R15-Pad1): track 0.00 -> 1.85 mm
- net CS11_A: track 0.00 -> 1.37 mm

Commit message: connected sw side of u5
Parts:
- added H3: PCB Common Earth, MountingHole:MountingHole_3.5mm_Pad_TopBottom, F.Cu at (293.4, 6.99)
- moved D1 1.27 mm to (17.2, 17.4)
- moved R16 0.76 mm to (30.6, 25.1), turned to 270 degrees
Connections:
- R16 pad 1: Net-(R16-Pad1) -> +3V3
- R16 pad 2: GND -> Net-(R16-Pad2)
- R19 pad 1: Net-(R19-Pad1) -> +3V3
- R19 pad 2: GND -> Net-(R19-Pad2)
- U5 pad 46: Net-(R16-Pad1) -> Net-(R16-Pad2)
- U6 pad 46: Net-(R19-Pad1) -> Net-(R19-Pad2)
Routing:
- net SW3_A: track 375.0 -> 453.9 mm
- net SW2_A: track 373.3 -> 451.2 mm
- net SW1_A: track 373.0 -> 448.4 mm
- net SW6_A: track 285.8 -> 354.5 mm, vias 0 -> 2
- net SW5_A: track 285.8 -> 351.4 mm, vias 0 -> 2
- net SW4_A: track 285.8 -> 347.9 mm, vias 0 -> 2
- net SW9_A: track 274.3 -> 300.0 mm, vias 0 -> 1
- net SW8_A: track 274.4 -> 298.0 mm, vias 0 -> 1
- net SW7_A: track 274.4 -> 297.6 mm, vias 0 -> 1
- net SW10_A: track 300.9 -> 323.3 mm
- net SW11_A: track 300.7 -> 322.1 mm
- net GND: track 3.09 -> 17.9 mm
- net SW12_A: track 299.9 -> 310.9 mm
- net Net-(R16-Pad1): track 4.25 -> 0.00 mm
- net Net-(R16-Pad2): track 0.00 -> 3.51 mm
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
Commit message: almost done with LER driver u5
Parts:
- moved J3 4.04 mm to (301.5, 26.9), turned to 270 degrees
- moved J2 2.82 mm to (307.3, 26.8)
- moved R9 2.09 mm to (347.2, 25.5), turned to 90 degrees
- moved R10 2.05 mm to (347.2, 22.5)
- moved C14 1.62 mm to (33.9, 11.4)
- moved C13 1.62 mm to (32.4, 11.4)
- moved C17 0.68 mm to (42.4, 16.5)
- moved C11 0.64 mm to (33.9, 25.1)
- moved C12 0.64 mm to (32.3, 25.1)
- moved R16 0.57 mm to (30.1, 24.9), turned to 90 degrees
- moved C16 0.52 mm to (39.0, 17.5)
- moved C15 0.51 mm to (37.3, 17.5)
- moved H3 0.28 mm to (293.1, 7.11)
Routing:
- net I2C_SCL: track 0.00 -> 328.3 mm, vias 0 -> 2
- net I2C_SDA: track 0.00 -> 327.1 mm, vias 0 -> 2
- net CS2_A: track 0.00 -> 136.1 mm, vias 0 -> 1
- net CS1_A: track 0.00 -> 108.2 mm, vias 0 -> 1
- net CS4_A: track 0.00 -> 70.5 mm, vias 0 -> 1
- net CS3_A: track 0.00 -> 51.8 mm, vias 0 -> 1
- net +3V3: track 0.00 -> 48.4 mm
- net CS5_A: track 0.00 -> 27.7 mm, vias 0 -> 1
- net CS6_A: track 0.00 -> 26.8 mm, vias 0 -> 1
- net CS7_A: track 0.00 -> 26.0 mm, vias 0 -> 1
- net CS8_A: track 0.00 -> 25.2 mm, vias 0 -> 1
- net CS9_A: track 0.00 -> 24.3 mm, vias 0 -> 1
- net CS10_A: track 0.00 -> 23.9 mm, vias 0 -> 1
- net CS12_A: track 0.00 -> 23.8 mm, vias 0 -> 1
- net CS11_A: track 0.00 -> 23.8 mm, vias 0 -> 1
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- added copper zone on B.Cu, net GND

Commit message: Updated LED Driver Footprint to have termal vias
Parts:
- U5, U6: footprint Lumissil:IS31FL3733B-QFLS4-TR -> Package_DFN_QFN:QFN-48-1EP_6x6mm_P0.4mm_EP4.2x4.2mm_ThermalVias

Commit message: Picked the actual correct footprint for the LED drivers
Parts:
- U5, U6: footprint Package_DFN_QFN:QFN-48-1EP_6x6mm_P0.4mm_EP4.2x4.2mm_ThermalVias -> Package_DFN_QFN:QFN-48-1EP_6x6mm_P0.4mm_EP4.6x4.6mm_ThermalVias

Commit message: led csa in progress
ledm csa in progress
Parts:
- moved J3 2.11 mm to (300.4, 28.7)
- moved J2 1.65 mm to (306.7, 28.3)
Routing:
- net (no net): track 0.00 -> 240.5 mm
- net CS12_A: track 23.8 -> 192.1 mm, vias 1 -> 2
- net CS11_A: track 23.8 -> 159.3 mm, vias 1 -> 2
- net CS6_A: track 26.8 -> 135.2 mm, vias 1 -> 3
- net CS10_A: track 23.9 -> 125.9 mm, vias 1 -> 2
- net CS5_A: track 27.7 -> 112.7 mm, vias 1 -> 3
- net CS9_A: track 24.3 -> 97.6 mm, vias 1 -> 2
- net CS7_A: track 26.0 -> 99.1 mm, vias 1 -> 2
- net CS8_A: track 25.2 -> 88.9 mm, vias 1 -> 2
- net CS4_A: track 70.5 -> 65.0 mm
- net I2C_SCL: track 328.3 -> 329.4 mm, vias 2 -> 3
- net I2C_SDA: track 327.1 -> 327.0 mm, vias 2 -> 3

Commit message: started led driver 2
Routing:
- net GND: track 17.9 -> 258.5 mm
- net (no net): track 240.5 -> 0.00 mm
- net CS10_A: track 125.9 -> 230.4 mm, vias 2 -> 3
- net CS9_A: track 97.6 -> 196.9 mm, vias 2 -> 3
- net CS8_A: track 88.9 -> 176.3 mm, vias 2 -> 3
- net CS11_A: track 159.3 -> 242.4 mm, vias 2 -> 3
- net CS12_A: track 192.1 -> 265.5 mm, vias 2 -> 3
- net CS7_A: track 99.1 -> 162.6 mm, vias 2 -> 3
- net CS1_B: track 0.00 -> 50.7 mm
- net CS2_B: track 0.00 -> 45.9 mm
- net CS3_B: track 0.00 -> 41.2 mm
- net SW9_A: track 300.0 -> 338.1 mm
- net SW8_A: track 298.0 -> 336.1 mm
- net SW7_A: track 297.6 -> 335.7 mm
- net CS5_B: track 0.00 -> 28.9 mm
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