File: 694210101R1/694210101R1.kicad_pcb (KiCad board)
At the start: 2 copper layers, 439.4 x 518.6 mm, 364 parts, among them J1 USB4085-GF-A, J2 Conn_01x02_Male, J3 Conn_01x02_Male, SW1 MX_SW, SW10 MX_SW, SW100 MX_SW, SW101 MX_SW, SW102 MX_SW, SW11 MX_SW, SW12 MX_SW, SW13 MX_SW, SW14 MX_SW, SW15 MX_SW, SW16 MX_SW, SW17 MX_SW, SW18 MX_SW, SW19 MX_SW, SW2 MX_SW, SW20 MX_SW, SW21 MX_SW, SW22 MX_SW, SW23 MX_SW, SW24 MX_SW, SW25 MX_SW, SW26 MX_SW, SW27 MX_SW, SW28 MX_SW, SW29 MX_SW, SW3 MX_SW, SW30 MX_SW, SW31 MX_SW, SW32 MX_SW, SW33 MX_SW, SW34 MX_SW, SW35 MX_SW, SW36 MX_SW, SW37 MX_SW, SW38 MX_SW, SW39 MX_SW, SW4 MX_SW, SW40 MX_SW, SW41 MX_SW, SW42 MX_SW, SW43 MX_SW, SW44 MX_SW, SW45 MX_SW, SW46 MX_SW, SW47 MX_SW, SW48 MX_SW, SW49 MX_SW, SW5 MX_SW, SW50 MX_SW, SW51 MX_SW, SW52 MX_SW, SW53 MX_SW, SW54 MX_SW, SW55 MX_SW, SW56 MX_SW, SW57 MX_SW, SW58 MX_SW, SW59 MX_SW, SW6 MX_SW, SW60 MX_SW, SW61 MX_SW, SW62 MX_SW, SW63 MX_SW, SW64 MX_SW, SW65 MX_SW, SW66 MX_SW, SW67 MX_SW, SW68 MX_SW, SW69 MX_SW, SW7 MX_SW, SW70 MX_SW, SW71 MX_SW, SW72 MX_SW, SW73 MX_SW, SW74 MX_SW, SW75 MX_SW, SW76 MX_SW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

Commit message: fixed file names, added additional source
Parts:
- removed the C23 at (717.6, 195.1)
- C10: renamed from C9; value CL10B104KB8NNNL -> CL10B474KA8NFNC
- C12: renamed from C13; value CL10B474KA8NFNC -> CL10B104KB8NNNL
- C16: renamed from C22; value CL10B104KB8NNNL -> TAJB226K016RNJ
- C19: renamed from C16; value TAJB226K016RNJ -> CL10B104KB8NNNL
- C21: renamed from C19; value CL10B104KB8NNNL -> CL10B474KA8NFNC
- C22: renamed from C15; value TAJB226K016RNJ -> CL10B104KB8NNNL
- U2: renamed from U1; value SOT-223_DIO -> AP2114HA-3.3TRG1
- U4, U5: value QFN-48_ISI -> IS31FL3733B-QFLS4-TR
- moved C10 632.5 mm to (85.9, 182.0)
- moved C16 632.5 mm to (43.9, 188.0)
- moved C18 632.5 mm to (81.4, 192.2)
- moved C2 632.5 mm to (285.7, 59.7)
- moved C3 632.5 mm to (285.7, 56.9)
- moved C4 632.5 mm to (285.7, 54.0)
- moved C5 632.5 mm to (285.7, 51.1)
- moved C6 632.5 mm to (285.7, 48.3)
- moved C7 632.5 mm to (121.0, 166.4)
- moved C9 632.5 mm to (77.8, 198.3)
- moved D107 632.5 mm to (55.6, 198.8)
- moved D113 632.5 mm to (55.6, 195.4)
- moved D114 632.5 mm to (51.4, 198.8)
- moved D117 632.5 mm to (55.6, 192.0)
- moved D118 632.5 mm to (42.5, 210.4)
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- renumbered C10 to C11, C11 to C13, C21 to C18, C18 to C23, C12 to C9, U2 to U1
Connections:
- C10 pad 2: GND -> Net-(C10-Pad2)
- C11 pad 2: GND -> Net-(C10-Pad2)
- C12 pad 2: GND -> Net-(C10-Pad2)
- C13 pad 2: GND -> Net-(C10-Pad2)
- C14 pad 2: GND -> Net-(C10-Pad2)
- C15 pad 2: GND -> Net-(C10-Pad2)
- C16 pad 2: GND -> Net-(C10-Pad2)
- C17 pad 2: GND -> Net-(C10-Pad2)
- C18 pad 2: GND -> Net-(C10-Pad2)
- C19 pad 2: GND -> Net-(C10-Pad2)
- C20 pad 2: GND -> Net-(C10-Pad2)
- C21 pad 2: GND -> Net-(C10-Pad2)
- C22 pad 2: GND -> Net-(C10-Pad2)
- C23 pad 2: GND -> Net-(C10-Pad2)
- C8 pad 2: GND -> Net-(C10-Pad2)
- C9 pad 2: GND -> Net-(C10-Pad2)
Other:
- board outline removed
