File: 694210101R1/694210101R1.sch (KiCad schematic (older format))
At the start: 226 parts, among them J1 USB4085-GF-A, J2 Conn_01x02_Male, J3 Conn_01x02_Male, SW1 MX_SW, SW10 MX_SW, SW100 MX_SW, SW101 MX_SW, SW102 MX_SW, SW11 MX_SW, SW12 MX_SW, SW13 MX_SW, SW14 MX_SW, SW15 MX_SW, SW16 MX_SW, SW17 MX_SW, SW18 MX_SW, SW19 MX_SW, SW2 MX_SW, SW20 MX_SW, SW21 MX_SW, SW22 MX_SW, SW23 MX_SW, SW24 MX_SW, SW25 MX_SW, SW26 MX_SW, SW27 MX_SW, SW28 MX_SW, SW29 MX_SW, SW3 MX_SW, SW30 MX_SW, SW31 MX_SW, SW32 MX_SW, SW33 MX_SW, SW34 MX_SW, SW35 MX_SW, SW36 MX_SW, SW37 MX_SW, SW38 MX_SW, SW39 MX_SW, SW4 MX_SW, SW40 MX_SW, SW41 MX_SW, SW42 MX_SW, SW43 MX_SW, SW44 MX_SW, SW45 MX_SW, SW46 MX_SW, SW47 MX_SW, SW48 MX_SW, SW49 MX_SW, SW5 MX_SW, SW50 MX_SW, SW51 MX_SW, SW52 MX_SW, SW53 MX_SW, SW54 MX_SW, SW55 MX_SW, SW56 MX_SW, SW57 MX_SW, SW58 MX_SW, SW59 MX_SW, SW6 MX_SW, SW60 MX_SW, SW61 MX_SW, SW62 MX_SW, SW63 MX_SW, SW64 MX_SW, SW65 MX_SW, SW66 MX_SW, SW67 MX_SW, SW68 MX_SW, SW69 MX_SW, SW7 MX_SW, SW70 MX_SW, SW71 MX_SW, SW72 MX_SW, SW73 MX_SW, SW74 MX_SW, SW75 MX_SW, SW76 MX_SW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

Commit message: fixed file names, added additional source
Parts:
- renumbered U2 to U1, U1 to U2
Changed lines of the file:
@@
 	2400 8950 1850 8950
 $Comp
-L power:GND #PWR02
+L power:GND #PWR0101
 U 1 1 5FF3187D
 P 2500 9950
-F 0 "#PWR02" H 2500 9700 50  0001 C CNN
+F 0 "#PWR0101" H 2500 9700 50  0001 C CNN
 F 1 "GND" H 2505 9777 50  0000 C CNN
 F 2 "" H 2500 9950 50  0001 C CNN
@@
 Connection ~ 2400 6350
 $Comp
-L power:+5V #PWR01
+L power:+5V #PWR0102
 U 1 1 5FF35DFE
 P 2400 6000
-F 0 "#PWR01" H 2400 5850 50  0001 C CNN
+F 0 "#PWR0102" H 2400 5850 50  0001 C CNN
 F 1 "+5V" H 2415 6173 50  0000 C CNN
 F 2 "" H 2400 6000 50  0001 C CNN
@@
 	2500 6550 2500 7550
 $Comp
-L DI-LVO:AP2114HA-3.3TRG1 U1
+L DI-LVO:AP2114HA-3.3TRG1 U2
 U 1 1 5FF9E77D
 P 2950 9500
-F 0 "U1" H 4050 9887 60  0000 C CNN
+F 0 "U2" H 4050 9887 60  0000 C CNN
 F 1 "AP2114HA-3.3TRG1" H 4050 9781 60  0000 C CNN
 F 2 "DI-LVO:AP2114HA-3.3TRG1" H 4050 9740 60  0001 C CNN
@@
 $EndComp
 $Comp
-L power:+5V #PWR03
+L power:+5V #PWR0103
 U 1 1 5FFA23B6
 P 2950 9500
-F 0 "#PWR03" H 2950 9350 50  0001 C CNN
+F 0 "#PWR0103" H 2950 9350 50  0001 C CNN
 F 1 "+5V" H 2965 9673 50  0000 C CNN
 F 2 "" H 2950 9500 50  0001 C CNN
@@
 Connection ~ 5550 9600
 $Comp
-L power:+3V3 #PWR04
+L power:+3V3 #PWR0104
 U 1 1 60025455
 P 6450 9600
-F 0 "#PWR04" H 6450 9450 50  0001 C CNN
+F 0 "#PWR0104" H 6450 9450 50  0001 C CNN
 F 1 "+3V3" H 6465 9773 50  0000 C CNN
 F 2 "" H 6450 9600 50  0001 C CNN
@@
 Connection ~ 2950 9950
 $Comp
-L power:+3V3 #PWR08
+L power:+3V3 #PWR0105
 U 1 1 6002F4CC
 P 8950 5950
-F 0 "#PWR08" H 8950 5800 50  0001 C CNN
+F 0 "#PWR0105" H 8950 5800 50  0001 C CNN
 F 1 "+3V3" H 8965 6123 50  0000 C CNN
 F 2 "" H 8950 5950 50  0001 C CNN
@@
 $EndComp
 $Comp
-L MCU_ST_STM32L4:STM32L433RBTx U2
+L MCU_ST_STM32L4:STM32L433RBTx U1
 U 1 1 5FE7C7AF
 P 8950 8200
-F 0 "U2" H 9200 6350 50  0000 C CNN
+F 0 "U1" H 9200 6350 50  0000 C CNN
 F 1 "STM32L433RBTx" H 9450 6250 50  0000 C CNN
 F 2 "Package_QFP:LQFP-64_10x10mm_P0.5mm" H 8350 6500 50  0001 R CNN
@@
 Connection ~ 8950 10100
 $Comp
-L power:GND #PWR07
+L power:GND #PWR0106
 U 1 1 5FFAF2AA
 P 8850 10200
-F 0 "#PWR07" H 8850 9950 50  0001 C CNN
+F 0 "#PWR0106" H 8850 9950 50  0001 C CNN
 F 1 "GND" H 8772 10163 50  0000 R CNN
 F 2 "" H 8850 10200 50  0001 C CNN
@@
 $EndComp
 $Comp
-L power:+3V3 #PWR06
+L power:+3V3 #PWR0107
 U 1 1 60076D41
 P 7700 7800
-F 0 "#PWR06" H 7700 7650 50  0001 C CNN
+F 0 "#PWR0107" H 7700 7650 50  0001 C CNN
 F 1 "+3V3" H 7715 7973 50  0000 C CNN
 F 2 "" H 7700 7800 50  0001 C CNN
@@
 	8250 6600 7950 6600
 $Comp
-L power:GND #PWR05
+L power:GND #PWR0108
 U 1 1 6007927B
 P 7550 6950
-F 0 "#PWR05" H 7550 6700 50  0001 C CNN
+F 0 "#PWR0108" H 7550 6700 50  0001 C CNN
 F 1 "GND" H 7555 6777 50  0000 C CNN
 F 2 "" H 7550 6950 50  0001 C CNN
@@
 $EndComp
 $Comp
-L power:+3V3 #PWR011
+L power:+3V3 #PWR0109
 U 1 1 5FEB4721
 P 15750 6350
-F 0 "#PWR011" H 15750 6200 50  0001 C CNN
+F 0 "#PWR0109" H 15750 6200 50  0001 C CNN
 F 1 "+3V3" H 15765 6523 50  0000 C CNN
 F 2 "" H 15750 6350 50  0001 C CNN
@@
 	10950 8000 10950 8050
 $Comp
-L power:+3V3 #PWR09
+L power:+3V3 #PWR0110
 U 1 1 60025E0E
 P 10750 8000
-F 0 "#PWR09" H 10750 7850 50  0001 C CNN
+F 0 "#PWR0110" H 10750 7850 50  0001 C CNN
 F 1 "+3V3" H 10765 8173 50  0000 C CNN
 F 2 "" H 10750 8000 50  0001 C CNN
@@
 Connection ~ 13500 8150
 $Comp
-L power:GND #PWR010
+L power:GND #PWR0111
 U 1 1 5FEB2ECC
 P 13500 8150
-F 0 "#PWR010" H 13500 7900 50  0001 C CNN
+F 0 "#PWR0111" H 13500 7900 50  0001 C CNN
 F 1 "GND" H 13505 7977 50  0000 C CNN
 F 2 "" H 13500 8150 50  0001 C CNN
@@
 S 13750 5500 900  800
 U 63A35802
-F0 "694200101R1_sheet_2" 50
-F1 "694200101R1_sheet_2.sch" 50
+F0 "694210101R1_sheet_2" 50
+F1 "694210101R1_sheet_2.sch" 50
 F2 "I2C_SDA" I L 13750 6100 50
 F3 "I2C_SCL" I L 13750 6000 50
