File: 694210101R1/694210101R1_sheet_2.sch (KiCad schematic (older format))
At the start: 89 parts, among them U3 M24M02-DRMN6TP, U4 IS31FL3733B-QFLS4-TR, U5 IS31FL3733B-QFLS4-TR

Commit message: fixed file names, added additional source
Parts:
- renumbered C14 to C12, C12 to C13, C15 to C14, C8 to C15, C23 to C16, C18 to C17, C22 to C18, C17 to C19, C21 to C20, C20 to C21, C16 to C22, C19 to C23, C9 to C8, C13 to C9
Connections:
- net CS14_A: no longer D160.2, D160.4, D160.6, D161.2, D161.4, D161.6, D162.2, D162.4, D162.6, D163.2, D163.4, D163.6, D164.2, D164.4, D164.6, D165.2, D165.4, D165.6, D166.2, D166.4, D166.6, D167.2, D167.4, D167.6
- net CS15_A: now also D160.2, D160.4, D160.6, D161.2, D161.4, D161.6, D162.2, D162.4, D162.6, D163.2, D163.4, D163.6
- net CS16_A: now also D164.2, D164.4, D164.6, D165.2, D165.4, D165.6, D166.2, D166.4, D166.6, D167.2, D167.4, D167.6
- net GND: no longer C10.2, C11.2, C12.2, C13.2, C14.2, C15.2, C16.2, C17.2, C18.2, C19.2, C20.2, C21.2, C22.2, C23.2, C8.2, C9.2
- new net: C10.2, C11.2, C12.2, C13.2, C14.2, C15.2, C16.2, C17.2, C18.2, C19.2, C20.2, C21.2, C22.2, C23.2, C8.2, C9.2
Other:
- moved on the sheet: C10, C11, C12, C13, C14, C15, C16, C17, C18, C19, C20, C21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
