File: 694200101R2/694200101R2.sch (KiCad schematic (older format))
At the start: 264 parts, among them J1 USB_C_Receptacle_USB2.0, J2 Conn_01x06_Male, SW1 MX_SW, SW10 MX_SW, SW100 MX_SW, SW101 MX_SW, SW102 MX_SW, SW103 MX_SW, SW104 MX_SW, SW105 MX_SW, SW106 MX_SW, SW107 MX_SW, SW108 SW_SPST, SW109 SW_SPDT, SW11 MX_SW, SW12 MX_SW, SW13 MX_SW, SW14 MX_SW, SW15 MX_SW, SW16 MX_SW, SW17 MX_SW, SW18 MX_SW, SW19 MX_SW, SW2 MX_SW, SW20 MX_SW, SW21 MX_SW, SW22 MX_SW, SW23 MX_SW, SW24 MX_SW, SW25 MX_SW, SW26 MX_SW, SW27 MX_SW, SW28 MX_SW, SW29 MX_SW, SW3 MX_SW, SW30 MX_SW, SW31 MX_SW, SW32 MX_SW, SW33 MX_SW, SW34 MX_SW, SW35 MX_SW, SW36 MX_SW, SW37 MX_SW, SW38 MX_SW, SW39 MX_SW, SW4 MX_SW, SW40 MX_SW, SW41 MX_SW, SW42 MX_SW, SW43 MX_SW, SW44 MX_SW, SW45 MX_SW, SW46 MX_SW, SW47 MX_SW, SW48 MX_SW, SW49 MX_SW, SW5 MX_SW, SW50 MX_SW, SW51 MX_SW, SW52 MX_SW, SW53 MX_SW, SW54 MX_SW, SW55 MX_SW, SW56 MX_SW, SW57 MX_SW, SW58 MX_SW, SW59 MX_SW, SW6 MX_SW, SW60 MX_SW, SW61 MX_SW, SW62 MX_SW, SW63 MX_SW, SW64 MX_SW, SW65 MX_SW, SW66 MX_SW, SW67 MX_SW, SW68 MX_SW, SW69 MX_SW, SW7 MX_SW, SW70 MX_SW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

Commit message: Removed rest of global labels
Connections:
- net D+: now reaches J1.A6 (D+), J1.B6 (D+), U2.4 (I/O2)
- net D-: now reaches J1.A7 (D-), J1.B7 (D-), U2.6 (I/O1)
Changed lines of the file:
@@
 	1    0    0    -1
 $EndComp
-Text GLabel 1350 850  1    50   Input ~ 0
-COL_0
 Wire Wire Line
 	1350 850  1350 900
@@
 Wire Wire Line
 	900  3150 900  3250
-Text GLabel 1950 850  1    50   Input ~ 0
-COL_1
 Wire Wire Line
 	1550 3500 1500 3500
@@
 Wire Wire Line
 	2600 900  2600 850
-Text GLabel 2600 850  1    50   Input ~ 0
-COL_2
 $Comp
 L cldg:MX_SW SW10
@@
 	2150 1300 2850 1300
 Connection ~ 2150 1300
-Text GLabel 3300 850  1    50   Input ~ 0
-COL_3
 Wire Wire Line
 	3300 850  3300 900
@@
 Wire Wire Line
 	4000 900  4000 850
-Text GLabel 4000 850  1    50   Input ~ 0
-COL_4
 $Comp
 L cldg:MX_SW SW21
@@
 Wire Wire Line
 	4700 900  4700 850
-Text GLabel 4700 850  1    50   Input ~ 0
-COL_5
 $Comp
 L cldg:MX_SW SW26
@@
 Wire Wire Line
 	5000 1550 4950 1550
-Text GLabel 5400 850  1    50   Input ~ 0
-COL_6
 Wire Wire Line
 	4250 1950 4950 1950
@@
 	1    0    0    -1
 $EndComp
-Text GLabel 6100 850  1    50   Input ~ 0
-COL_7
 Wire Wire Line
 	6100 900  6100 850
@@
 Wire Wire Line
 	6800 850  6800 900
-Text GLabel 6800 850  1    50   Input ~ 0
-COL_8
 Wire Wire Line
 	6350 1200 6350 1300
@@
 Wire Wire Line
 	16050 850  16050 1550
-Text GLabel 16050 850  1    50   Input ~ 0
-COL_22
 Wire Wire Line
 	15650 1550 15600 1550
@@
 Wire Wire Line
 	15300 850  15300 900
-Text GLabel 15300 850  1    50   Input ~ 0
-COL_21
 Connection ~ 14150 1300
 Wire Wire Line
@@
 Wire Wire Line
 	13450 1300 14150 1300
-Text GLabel 14600 850  1    50   Input ~ 0
-COL_20
 Wire Wire Line
 	14600 900  14600 850
@@
 	1    0    0    -1
 $EndComp
-Text GLabel 13900 850  1    50   Input ~ 0
-COL_19
 Connection ~ 12750 1300
 Wire Wire Line
@@
 Wire Wire Line
 	12050 1300 12750 1300
-Text GLabel 13200 850  1    50   Input ~ 0
-COL_17
 Wire Wire Line
 	13200 900  13200 850
@@
 Wire Wire Line
 	11350 1300 12050 1300
-Text GLabel 12500 850  1    50   Input ~ 0
-COL_16
 Wire Wire Line
 	12500 900  12500 850
@@
 	1    0    0    -1
 $EndComp
-Text GLabel 11800 850  1    50   Input ~ 0
-COL_15
 Wire Wire Line
 	11800 900  11800 850
@@
 	1    0    0    -1
 $EndComp
-Text GLabel 11050 850  1    50   Input ~ 0
-COL_14
 Wire Wire Line
 	11050 900  11050 850
@@
 	1    0    0    -1
 $EndComp
-Text GLabel 10350 850  1    50   Input ~ 0
-COL_13
 Wire Wire Line
 	9900 1200 9900 1300
@@
 	1    0    0    -1
 $EndComp
-Text GLabel 9650 850  1    50   Input ~ 0
-COL_12
 Wire Wire Line
 	9650 900  9650 850
@@
 	1    0    0    -1
 $EndComp
-Text GLabel 8950 850  1    50   Input ~ 0
-COL_11
 Wire Wire Line
 	8950 900  8950 850
@@
 Wire Wire Line
 	7050 1300 7750 1300
-Text GLabel 8200 850  1    50   Input ~ 0
-COL_10
 Wire Wire Line
 	8200 900  8200 850
@@
 	1    0    0    -1
 $EndComp
-Text GLabel 7500 850  1    50   Input ~ 0
-COL_9
 Wire Wire Line
 	7500 900  7500 850
@@
 Wire Wire Line
 	5500 8000 5650 8000
-Text GLabel 5650 8000 2    50   Input ~ 0
-SWCLK
 Wire Wire Line
 	5500 8100 6000 8100
@@
 Wire Wire Line
 	5500 8200 5650 8200
-Text GLabel 5650 8200 2    50   Input ~ 0
-SWDIO
 Wire Wire Line
 	5900 8300 5500 8300
 Wire Wire Line
 	5500 8400 5650 8400
-Text GLabel 5650 8400 2    50   Input ~ 0
-SWO
 Wire Wire Line
 	5900 8700 5900 8750
@@
 	1    0    0    -1
 $EndComp
-Text Label 5900 8450 0    50   ~ 0
+Text Label 6050 8450 0    50   ~ 0
 RST
 Wire Wire Line
@@
 	-1   0    0    -1
 $EndComp
-Text GLabel 4350 5800 2    50   Input ~ 0
-USB_D-
-Text GLabel 4350 6200 2    50   Input ~ 0
-USB_D+
 NoConn ~ 1750 6550
 NoConn ~ 1750 6450
@@
 Wire Wire Line
 	5900 8450 5900 8500
-Text GLabel 6050 8450 2    50   Input ~ 0
-RST
 Text Notes 5100 8650 0    50   ~ 0
 JTAG/RST
@@
 Text Notes 4850 7300 0    50   ~ 0
 Stabs and Mounting Holes
-Text GLabel 10775 7175 2    50   Input ~ 0
-SWDIO
-Text GLabel 10775 6275 2    50   Input ~ 0
-COL_22
-Text GLabel 9375 5875 0    50   Input ~ 0
-RST
 $Comp
 L Resistor-Lib:RMCF0805FT510R R5
@@
 Wire Wire Line
 	8050 5200 8000 5200
-Text GLabel 10775 7875 2    50   Input ~ 0
-SWO
-Text GLabel 10775 7275 2    50   Input ~ 0
-SWCLK
-Text GLabel 10775 6375 2    50   Input ~ 0
-COL_21
-Text GLabel 10775 6475 2    50   Input ~ 0
-COL_20
-Text GLabel 10775 6575 2    50   Input ~ 0
-COL_19
-Text GLabel 9375 7875 0    50   Input ~ 0
-COL_17
-Text GLabel 9375 7975 0    50   Input ~ 0
-COL_16
-Text GLabel 9375 8075 0    50   Input ~ 0
-COL_15
-Text GLabel 10775 7775 2    50   Input ~ 0
-COL_14
-Text GLabel 10775 8575 2    50   Input ~ 0
-COL_13
-Text GLabel 10775 8675 2    50   Input ~ 0
-COL_12
-Text GLabel 10775 8775 2    50   Input ~ 0
-COL_11
-Text GLabel 10775 8875 2    50   Input ~ 0
-COL_10
-Text GLabel 10775 8975 2    50   Input ~ 0
-COL_9
-Text GLabel 10775 9075 2    50   Input ~ 0
-COL_8
-Text GLabel 9375 8175 0    50   Input ~ 0
-COL_7
-Text GLabel 9375 8275 0    50   Input ~ 0
-COL_6
-Text GLabel 9375 8375 0    50   Input ~ 0
-COL_5
-Text GLabel 9375 8475 0    50   Input ~ 0
-COL_4
-Text GLabel 10775 6675 2    50   Input ~ 0
-COL_3
-Text GLabel 10775 6775 2    50   Input ~ 0
-COL_2
-Text GLabel 10775 6875 2    50   Input ~ 0
-COL_1
-Text GLabel 10775 7375 2    50   Input ~ 0
-COL_0
 $Comp
 L power:+3V3 #PWR014
@@
 	1    0    0    -1
 $EndComp
-Text GLabel 10775 7675 2    50   Input ~ 0
-ENCODER_B
-Text GLabel 10775 7575 2    50   Input ~ 0
-ENCODER_A
-Text GLabel 10775 6975 2    50   Input ~ 0
-USB_D-
-Text GLabel 10775 7075 2    50   Input ~ 0
-USB_D+
 Wire Wire Line
 	10025 9375 10025 9475
@@
 	-1   0    0    -1
 $EndComp
-Text GLabel 12400 6125 0    50   Input ~ 0
-ENCODER_B
-Text GLabel 12400 5925 0    50   Input ~ 0
-ENCODER_A
 Text Notes 11725 7325 0    50   ~ 0
 Encoder
@@
 Wire Wire Line
 	13175 6225 13100 6225
-Text GLabel 13725 5825 2    50   Input ~ 0
-COL_22
 $Comp
 L power:GND #PWR015
@@
 	9375 7075 9425 7075
 Wire Wire Line
-	9375 6975 9425 6975
-Wire Wire Line
 	9425 7375 9375 7375
 Wire Wire Line
@@
 Text Label 1850 9075 2    50   ~ 0
 OSC_OUT
-Text Label 9375 6975 2    50   ~ 0
-OSC_IN
 Text Label 2850 9075 0    50   ~ 0
 OSC_IN
@@
 	1    0    0    -1
 $EndComp
+Text Label 10775 6875 0    50   ~ 0
+COL_1
+Text Label 10775 6775 0    50   ~ 0
+COL_2
+Text Label 10775 6675 0    50   ~ 0
+COL_3
+Text Label 10775 6575 0    50   ~ 0
+COL_19
+Text Label 10775 6475 0    50   ~ 0
+COL_20
+Text Label 10775 6375 0    50   ~ 0
+COL_21
+Text Label 10775 6275 0    50   ~ 0
+COL_22
+Text Label 9375 8475 2    50   ~ 0
+COL_4
+Text Label 9375 8375 2    50   ~ 0
+COL_5
+Text Label 9375 8275 2    50   ~ 0
+COL_6
+Text Label 9375 8175 2    50   ~ 0
+COL_7
+Text Label 9375 8075 2    50   ~ 0
+COL_15
+Text Label 9375 7975 2    50   ~ 0
+COL_16
+Text Label 9375 7875 2    50   ~ 0
+COL_17
+Text Label 10775 9075 0    50   ~ 0
+COL_8
+Text Label 10775 8975 0    50   ~ 0
+COL_9
+Text Label 10775 8875 0    50   ~ 0
+COL_10
+Text Label 10775 8775 0    50   ~ 0
+COL_11
+Text Label 10775 8675 0    50   ~ 0
+COL_12
+Text Label 10775 8575 0    50   ~ 0
+COL_13
+Text Label 2500 5800 0    50   ~ 0
+D-
+Text Label 2525 6200 0    50   ~ 0
+D+
+Text Label 1950 850  1    50   ~ 0
+COL_1
+Text Label 10775 7775 0    50   ~ 0
+COL_14
+Text Label 10775 7375 0    50   ~ 0
+COL_0
+Text Label 9375 5875 2    50   ~ 0
+RST
+Text Label 1350 850  1    50   ~ 0
+COL_0
+Text Label 2600 850  1    50   ~ 0
+COL_2
+Text Label 3300 850  1    50   ~ 0
+COL_3
+Text Label 4000 850  1    50   ~ 0
+COL_4
+Text Label 4700 850  1    50   ~ 0
+COL_5
+Text Label 5400 850  1    50   ~ 0
+COL_6
+Text Label 6100 850  1    50   ~ 0
+COL_7
+Text Label 6800 850  1    50   ~ 0
+COL_8
+Text Label 7500 850  1    50   ~ 0
+COL_9
+Text Label 8200 850  1    50   ~ 0
+COL_10
+Text Label 8950 850  1    50   ~ 0
+COL_11
+Text Label 9650 850  1    50   ~ 0
+COL_12
+Text Label 10350 850  1    50   ~ 0
+COL_13
+Text Label 11050 850  1    50   ~ 0
+COL_14
+Text Label 11800 850  1    50   ~ 0
+COL_15
+Text Label 12500 850  1    50   ~ 0
+COL_16
+Text Label 13200 850  1    50   ~ 0
+COL_17
+Text Label 13900 850  1    50   ~ 0
+COL_19
+Text Label 14600 850  1    50   ~ 0
+COL_20
+Text Label 15300 850  1    50   ~ 0
+COL_21
+Text Label 16050 850  1    50   ~ 0
+COL_22
+Text Label 13725 5825 0    50   ~ 0
+COL_22
+Text Label 10775 7675 0    50   ~ 0
+ENCODER_B
+Text Label 10775 7575 0    50   ~ 0
+ENCODER_A
+Text Label 12400 6125 2    50   ~ 0
+ENCODER_B
+Text Label 12400 5925 2    50   ~ 0
+ENCODER_A
+Text Label 10775 7875 0    50   ~ 0
+SWO
+Text Label 10775 7275 0    50   ~ 0
+SWCLK
+Text Label 10775 7175 0    50   ~ 0
+SWDIO
+Text Label 5650 8400 0    50   ~ 0
+SWO
+Text Label 5650 8200 0    50   ~ 0
+SWDIO
+Text Label 5650 8000 0    50   ~ 0
+SWCLK
+Text Label 10775 7075 0    50   ~ 0
+USB_D+
+Text Label 10775 6975 0    50   ~ 0
+USB_D-
+Text Label 4350 6200 0    50   ~ 0
+USB_D+
+Text Label 4350 5800 0    50   ~ 0
+USB_D-
+Wire Wire Line
+	9375 6975 9425 6975
+Text Label 9375 6975 2    50   ~ 0
+OSC_IN
 $EndSCHEMATC

Commit message: Updated Footprints to have CAD Models
Need footprints on board to allow for case modifications
Parts:
- ENC1: footprint digikey-footprints:Rotary_Encoder_Switched_PEC11R -> cldg:Rotary_Encoder_Switched_PEC11R
- J1: footprint Connector_USB:USB_C_Receptacle_GCT_USB4085 -> cldg:USB_C_Receptacle_GCT_USB4085
- SW109: footprint Button_Switch_SMD:SW_SPDT_CK-JS102011SAQN -> cldg:SW_SPDT_CK-JS102011SAQN
- U1: footprint digikey-footprints:SOT-223 -> Package_TO_SOT_SMD:SOT-223
- U4: footprint Package_SO:SO-8_3.9x4.9mm_P1.27mm -> Package_SO:SOIC-8_3.9x4.9mm_P1.27mm
Changed lines of the file:
@@
 F 0 "J1" H 1257 6817 50  0000 C CNN
 F 1 "USB_C_Receptacle_USB2.0" H 1257 6726 50  0000 C CNN
-F 2 "Connector_USB:USB_C_Receptacle_GCT_USB4085" H 1300 5950 50  0001 C CNN
+F 2 "cldg:USB_C_Receptacle_GCT_USB4085" H 1300 5950 50  0001 C CNN
 F 3 "https://www.usb.org/sites/default/files/documents/usb_type-c.zip" H 1300 5950 50  0001 C CNN
 	1    1150 5950
@@
 F 0 "ENC1" H 13400 6225 60  0000 C CNN
 F 1 "PEC11R-4215F-S0024" H 13800 6150 60  0000 C CNN
-F 2 "digikey-footprints:Rotary_Encoder_Switched_PEC11R" H 13675 6125 60  0001 L CNN
+F 2 "cldg:Rotary_Encoder_Switched_PEC11R" H 13675 6125 60  0001 L CNN
 F 3 "https://www.bourns.com/docs/Product-Datasheets/PEC11R.pdf" H 13675 6225 60  0001 L CNN
 F 4 "PEC11R-4215F-S0024-ND" H 13675 6325 60  0001 L CNN "Digi-Key_PN"
@@
 F 0 "SW109" H 7475 8685 50  0000 C CNN
 F 1 "SW_SPDT" H 7475 8594 50  0000 C CNN
-F 2 "Button_Switch_SMD:SW_SPDT_CK-JS102011SAQN" H 7475 8400 50  0001 C CNN
+F 2 "cldg:SW_SPDT_CK-JS102011SAQN" H 7475 8400 50  0001 C CNN
 F 3 "~" H 7475 8400 50  0001 C CNN
 	1    7475 8400
@@
 F 0 "U4" H 12700 8400 50  0000 C CNN
 F 1 "24LC512" H 12600 8325 50  0000 C CNN
-F 2 "Package_SO:SO-8_3.9x4.9mm_P1.27mm" H 12900 8075 50  0001 C CNN
+F 2 "Package_SO:SOIC-8_3.9x4.9mm_P1.27mm" H 12900 8075 50  0001 C CNN
 F 3 "http://ww1.microchip.com/downloads/en/DeviceDoc/21754M.pdf" H 12900 8075 50  0001 C CNN
 	1    12900 8075
@@
 F 0 "U1" H 2600 8062 60  0000 C CNN
 F 1 "AP2114HA-3_3TRG1" H 2600 7956 60  0000 C CNN
-F 2 "digikey-footprints:SOT-223" H 2850 7975 60  0001 L CNN
+F 2 "Package_TO_SOT_SMD:SOT-223" H 2850 7975 60  0001 L CNN
 F 3 "https://www.diodes.com/assets/Datasheets/AP2114.pdf" H 2850 8075 60  0001 L CNN
 F 4 "AP2114H-3.3TRG1DICT-ND" H 2850 8175 60  0001 L CNN "Digi-Key_PN"
