File: 694200101R2/694200101R2_sheet_2.sch (KiCad schematic (older format))
At the start: 76 parts, among them U5 IS31FL3733-TQ

Commit message: Fixed Ratsnest errors from prettifying schematic
Parts:
- renumbered R12 to R15, R13 to R16, R14 to R17
Changed lines of the file:
@@
 $EndComp
 $Comp
-L Device:R_US R13
+L Device:R_US R16
 U 1 1 64CF3D0D
 P 6300 7350
-F 0 "R13" V 6175 7525 50  0000 C CNN
+F 0 "R16" V 6175 7525 50  0000 C CNN
 F 1 "100k" V 6250 7525 50  0000 C CNN
 F 2 "Resistor_SMD:R_0603_1608Metric" V 6340 7340 50  0001 C CNN
@@
 $EndComp
 $Comp
-L Device:R_US R14
+L Device:R_US R17
 U 1 1 6954A924
 P 6325 7925
-F 0 "R14" H 6393 7971 50  0000 L CNN
+F 0 "R17" H 6393 7971 50  0000 L CNN
 F 1 "59k" H 6393 7880 50  0000 L CNN
 F 2 "Resistor_SMD:R_2512_6332Metric" V 6365 7915 50  0001 C CNN
@@
 $EndComp
 $Comp
-L Device:R_US R12
+L Device:R_US R15
 U 1 1 64C0E663
 P 6300 7450
-F 0 "R12" V 6250 7600 50  0000 C CNN
+F 0 "R15" V 6250 7600 50  0000 C CNN
 F 1 "100k" V 6175 7600 50  0000 C CNN
 F 2 "Resistor_SMD:R_0603_1608Metric" V 6340 7440 50  0001 C CNN

Commit message: Updated Footprints to have CAD Models
Need footprints on board to allow for case modifications
Parts:
- C17: footprint capacitor-lib:CAPPC3528X210N -> Capacitor_Tantalum_SMD:CP_EIA-3528-21_Kemet-B
Changed lines of the file:
@@
 F 0 "C17" H 9490 7221 50  0000 L CNN
 F 1 "22uF" H 9490 7130 50  0000 L CNN
-F 2 "capacitor-lib:CAPPC3528X210N" H 9375 7175 50  0001 C CNN
+F 2 "Capacitor_Tantalum_SMD:CP_EIA-3528-21_Kemet-B" H 9375 7175 50  0001 C CNN
 F 3 "~" H 9375 7175 50  0001 C CNN
 	1    9375 7175
